Commit message: Cleaned up some of the code to work on NRG magni, gazebo is still a bit broken

File: magni_description/urdf/magni_base.urdf.xacro (robot description, xacro)
@@ -5,5 +5,4 @@
   <xacro:property name="wheel_xpos" value="0.11" />
   <xacro:include filename="$(find magni_description)/urdf/magni.transmission.xacro" />
-  <xacro:include filename="$(find magni_description)/urdf/magni.gazebo.xacro" />
   <xacro:include filename="$(find magni_description)/urdf/inertial.xacro" />
   <!-- Robot base_link -->
@@ -116,10 +115,5 @@
   <ros2_control name="MagniSystem" type="system">
     <hardware>
-      <xacro:if value="$(arg use_sim)">
-        <plugin>gz_ros2_control/GazeboSimSystem</plugin>
-      </xacro:if>
-      <xacro:unless value="$(arg use_sim)">
-        <plugin>ubiquity_motor_ros2/MotorHardware</plugin>
-      </xacro:unless>
+      <plugin>ubiquity_motor_ros2/MotorHardware</plugin>
     </hardware>
     <joint name="left_wheel_joint">
