Commit message: Adding gazebo sim

File: magni_description/urdf/inertial.xacro (robot description, xacro)
@@ -25,5 +25,4 @@
 -->
 <robot xmlns:xacro="http://wiki.ros.org/xacro">
-    <xacro:property name="M_PI" value="3.1415926535897931" />
     <!-- see https://secure.wikimedia.org/wikipedia/en/wiki/List_of_moment_of_inertia_tensors -->
     <!-- #################### versions without origin #################### -->

File: magni_description/urdf/robot.urdf.xacro (robot description, xacro)
@@ -2,5 +2,6 @@
 <robot xmlns:xacro="http://wiki.ros.org/xacro" name="magni">
   <xacro:arg name="robot_type" default="gen_6_mini" />
+  <xacro:arg name="sim" default="false" />
   <xacro:include filename="$(find magni_description)/urdf/robots/$(arg robot_type).urdf.xacro" />
-  <xacro:magni />
+  <xacro:magni sim="$(arg sim)" />
 </robot>

File: magni_description/urdf/robots/gen_5_silver.urdf.xacro (robot description, xacro)
@@ -2,5 +2,5 @@
 <robot xmlns:xacro="http://wiki.ros.org/xacro">
   <xacro:macro name="magni"
-    params="prefix:='' sonars_installed:=true shell_installed:=false tower_installed:=false camera_extrinsics_file:='' lidar_extrinsics_file:=''">
+    params="prefix:='' sim:=false controller_config='$(find ubiquity_motor_ros2)/cfg/conf.yaml' sonars_installed:=true shell_installed:=false tower_installed:=false camera_extrinsics_file:='' lidar_extrinsics_file:=''">
     <xacro:property name="wheel_r" value="0.1" />
     <xacro:property name="wheel_xpos" value="0.11" />
@@ -16,16 +16,4 @@
         <geometry>
           <mesh filename="package://magni_description/meshes/gen5/chassis.dae" />
-        </geometry>
-      </visual>
-      <visual>
-        <origin xyz="${-wheel_xpos-0.169} 0.17 ${-wheel_r+0.09}" rpy="0 0 ${pi}" />
-        <geometry>
-          <mesh filename="package://magni_description/meshes/common/caster_wheel.dae" />
-        </geometry>
-      </visual>
-      <visual>
-        <origin xyz="${-wheel_xpos-0.169} -0.17 ${-wheel_r+0.09}" rpy="0 0 ${pi}" />
-        <geometry>
-          <mesh filename="package://magni_description/meshes/common/caster_wheel.dae" />
         </geometry>
       </visual>
@@ -162,4 +150,10 @@
     <xacro:macro name="caster_wheel" params="wheel_prefix reflect">
       <link name="${wheel_prefix}_caster_wheel">
+        <visual>
+          <origin xyz="${-wheel_xpos-0.169} ${reflect*0.17} ${-wheel_r+0.09}" rpy="0 0 ${pi}" />
+          <geometry>
+            <mesh filename="package://magni_description/meshes/common/caster_wheel.dae" />
+          </geometry>
+        </visual>
         <collision>
           <origin xyz="${-wheel_xpos-0.19} ${reflect*0.169} ${-wheel_r+0.04}" rpy="0 0 0" />
@@ -211,21 +205,47 @@
     </xacro:if>
     <!-- ROS 2 Control block -->
-    <ros2_control name="ubiquity_motor_ros2/MotorHardware" type="system">
-      <hardware>
-        <plugin>ubiquity_motor_ros2/MotorHardware</plugin>
-      </hardware>
-      <joint name="${prefix}left_wheel_joint">
-        <command_interface name="velocity" />
-        <state_interface name="position" />
-        <state_interface name="velocity" />
-        <state_interface name="effort" />
-      </joint>
-      <joint name="${prefix}right_wheel_joint">
-        <command_interface name="velocity" />
-        <state_interface name="position" />
-        <state_interface name="velocity" />
-        <state_interface name="effort" />
-      </joint>
-    </ros2_control>
+    <xacro:unless value="${sim}">
+      <ros2_control name="ubiquity_motor_ros2/MotorHardware" type="system">
+        <hardware>
+          <plugin>ubiquity_motor_ros2/MotorHardware</plugin>
+        </hardware>
+        <joint name="${prefix}left_wheel_joint">
+          <command_interface name="velocity" />
+          <state_interface name="position" />
+          <state_interface name="velocity" />
+          <state_interface name="effort" />
+        </joint>
+        <joint name="${prefix}right_wheel_joint">
+          <command_interface name="velocity" />
+          <state_interface name="position" />
+          <state_interface name="velocity" />
+          <state_interface name="effort" />
+        </joint>
+      </ros2_control>
+    </xacro:unless>
+    <xacro:if value="${sim}">
+      <ros2_control name="GazeboSimSystem" type="system">
+        <hardware>
+          <plugin>gz_ros2_control/GazeboSimSystem</plugin>
+        </hardware>
+        <joint name="${prefix}left_wheel_joint">
+          <command_interface name="velocity" />
+          <state_interface name="position" />
+          <state_interface name="velocity" />
+          <state_interface name="effort" />
+        </joint>
+        <joint name="${prefix}right_wheel_joint">
+          <command_interface name="velocity" />
+          <state_interface name="position" />
+          <state_interface name="velocity" />
+          <state_interface name="effort" />
+        </joint>
+      </ros2_control>
+      <gazebo>
+        <plugin filename="gz_ros2_control-system" name="gz_ros2_control::GazeboSimROS2ControlPlugin">
+          <parameters>${controller_config}</parameters>
+        </plugin>
+      </gazebo>
+    </xacro:if>
   </xacro:macro>
 </robot>
