Commit message: Fixing URDF files

File: magni_description/urdf/robots/gen_6_mini.urdf.xacro (robot description, xacro)
@@ -1,146 +1,148 @@
 <?xml version="1.0"?>
-<robot xmlns:xacro="http://wiki.ros.org/xacro" name="gen_6_mini">
-  <!-- Arguments -->
-  <xacro:arg name="use_sim" default="false"/>
-  <!-- Properties -->
-  <xacro:property name="wheel_r" value="0.1" />
-  <xacro:property name="wheel_xpos" value="0.11" />
-  <!-- Includes -->
-  <!-- <xacro:include filename="$(find magni_description)/urdf/magni.transmission.xacro" /> -->
-  <xacro:include filename="$(find magni_description)/urdf/magni.gazebo.xacro" />
-  <xacro:include filename="$(find magni_description)/urdf/inertial.xacro" />
-  <xacro:include filename="$(find magni_description)/urdf/sensors/ur_c1_lidar.xacro" />
-  <!-- Robot base_link -->
-  <link name="base_link">
-    <visual>
-      <origin xyz="${-wheel_xpos} 0 ${-wheel_r+0.071}" rpy="0 0 0" />
-      <geometry>
-        <mesh filename="package://magni_description/meshes/gen6/chassis_mini.dae" />
-      </geometry>
-    </visual>
-	<visual>
-      <origin xyz="${-wheel_xpos-0.169} 0.17 ${-wheel_r+0.09}" rpy="0 0 ${pi}" />
-      <geometry>
-        <mesh filename="package://magni_description/meshes/common/caster_wheel.dae" />
-      </geometry>
-    </visual>
-	<visual>
-      <origin xyz="${-wheel_xpos-0.169} -0.17 ${-wheel_r+0.09}" rpy="0 0 ${pi}" />
-      <geometry>
-        <mesh filename="package://magni_description/meshes/common/caster_wheel.dae" />
-      </geometry>
-    </visual>
-    <collision>
-	  <origin xyz="${-wheel_xpos} 0 ${-wheel_r+0.151}" rpy="0 0 0" />
-      <geometry>
-        <box size="0.398 0.268 0.160"/>
-      </geometry>
-    </collision>
-    <collision>
-      <origin xyz="${-wheel_xpos-0.026} 0 ${-wheel_r+0.248}" rpy="0 0 0" />
-      <geometry>
-        <box size="0.375 0.268 0.034"/>
-      </geometry>
-    </collision>
-    <collision>
-      <origin xyz="${-wheel_xpos-0.169} 0.169 ${-wheel_r+0.106}" rpy="0 0 0" />
-      <geometry>
-        <box size="0.1 0.07 0.07"/>
-      </geometry>
-    </collision>
-    <collision>
-      <origin xyz="${-wheel_xpos-0.169} -0.169 ${-wheel_r+0.106}" rpy="0 0 0" />
-      <geometry>
-        <box size="0.1 0.07 0.07"/>
-      </geometry>
-    </collision>
-    <xacro:box_inertial_with_origin  x="0.398" y="0.221" z="0.150" mass="10.0">
-      <origin xyz="-0.15 0 0.03" rpy="0 0 0" />
-    </xacro:box_inertial_with_origin>
-  </link>
-  <!-- Fixed offset from the floor to the center of the wheels -->
-  <link name="base_footprint"/>
-  <joint name="base_footprint_joint" type="fixed">
-    <parent link="base_footprint"/>
-    <child link="base_link"/>
-    <origin xyz="0 0 ${wheel_r}" rpy="0 0 0"/>
-  </joint>
-  <!-- Macro for defining wheels -->
-  <xacro:macro name="wheel" params="prefix reflect">
-    <link name="${prefix}_wheel">
+<robot xmlns:xacro="http://wiki.ros.org/xacro">
+  <xacro:macro name="magni">
+    <!-- Arguments -->
+    <xacro:arg name="use_sim" default="false" />
+    <!-- Properties -->
+    <xacro:property name="wheel_r" value="0.1" />
+    <xacro:property name="wheel_xpos" value="0.11" />
+    <!-- Includes -->
+    <!-- <xacro:include filename="$(find magni_description)/urdf/magni.transmission.xacro" /> -->
+    <!-- <xacro:include filename="$(find magni_description)/urdf/magni.gazebo.xacro" /> -->
+    <xacro:include filename="$(find magni_description)/urdf/inertial.xacro" />
+    <xacro:include filename="$(find magni_description)/urdf/sensors/ur_c1_lidar.xacro" />
+    <!-- Robot base_link -->
+    <link name="base_link">
       <visual>
-        <origin xyz="${-0.071*reflect} 0 0" rpy="0 ${(reflect-1)*pi/2} 0" />
+        <origin xyz="${-wheel_xpos} 0 ${-wheel_r+0.071}" rpy="0 0 0" />
         <geometry>
-          <mesh filename="package://magni_description/meshes/common/standard_wheel.dae" />
+          <mesh filename="package://magni_description/meshes/gen6/chassis_mini.dae" />
+        </geometry>
+      </visual>
+      <visual>
+        <origin xyz="${-wheel_xpos-0.169} 0.17 ${-wheel_r+0.09}" rpy="0 0 ${pi}" />
+        <geometry>
+          <mesh filename="package://magni_description/meshes/common/caster_wheel.dae" />
+        </geometry>
+      </visual>
+      <visual>
+        <origin xyz="${-wheel_xpos-0.169} -0.17 ${-wheel_r+0.09}" rpy="0 0 ${pi}" />
+        <geometry>
+          <mesh filename="package://magni_description/meshes/common/caster_wheel.dae" />
         </geometry>
       </visual>
       <collision>
-        <origin xyz="0 0 0" rpy="0 ${pi/2} 0" />
+        <origin xyz="${-wheel_xpos} 0 ${-wheel_r+0.151}" rpy="0 0 0" />
         <geometry>
-          <cylinder radius="${wheel_r}" length="0.05"/>
+          <box size="0.398 0.268 0.160" />
         </geometry>
       </collision>
       <collision>
-        <origin xyz="${0.033*reflect} 0 0" rpy="0 ${pi/2} 0" />
+        <origin xyz="${-wheel_xpos-0.026} 0 ${-wheel_r+0.248}" rpy="0 0 0" />
         <geometry>
-          <cylinder radius="0.064" length="0.016"/>
+          <box size="0.375 0.268 0.034" />
         </geometry>
       </collision>
-      <xacro:cylinder_inertial_with_origin radius="${wheel_r}" length="0.05" mass="3.34">
-        <origin xyz="0 0 0" rpy="0 ${pi/2} 0" />
-      </xacro:cylinder_inertial_with_origin>
-    </link>
-    <joint name="${prefix}_wheel_joint" type="continuous">
-      <axis xyz="1 0 0" rpy="0 0 0" />
-      <parent link="base_link"/>
-      <child link="${prefix}_wheel"/>
-      <origin xyz="0 ${0.163*reflect} 0" rpy="0 0 ${pi/2}"/>
-    </joint>
-  </xacro:macro>
-  <xacro:wheel prefix="left" reflect="1"/>
-  <xacro:wheel prefix="right" reflect="-1"/>
-  <!-- Macro for defining caster wheels -->
-  <xacro:macro name="caster_wheel" params="prefix reflect">
-    <link name="${prefix}_caster_wheel">
       <collision>
-        <origin xyz="${-wheel_xpos-0.19} ${reflect*0.169} ${-wheel_r+0.04}" rpy="0 0 0" />
+        <origin xyz="${-wheel_xpos-0.169} 0.169 ${-wheel_r+0.106}" rpy="0 0 0" />
         <geometry>
-          <sphere radius="0.04"/>
+          <box size="0.1 0.07 0.07" />
         </geometry>
       </collision>
+      <collision>
+        <origin xyz="${-wheel_xpos-0.169} -0.169 ${-wheel_r+0.106}" rpy="0 0 0" />
+        <geometry>
+          <box size="0.1 0.07 0.07" />
+        </geometry>
+      </collision>
+      <xacro:box_inertial_with_origin x="0.398" y="0.221" z="0.150" mass="10.0">
+        <origin xyz="-0.15 0 0.03" rpy="0 0 0" />
+      </xacro:box_inertial_with_origin>
     </link>
-    <joint name="${prefix}_caster_wheel_joint" type="fixed">
-      <parent link="base_link"/>
-      <child link="${prefix}_caster_wheel"/>
+    <!-- Fixed offset from the floor to the center of the wheels -->
+    <link name="base_footprint" />
+    <joint name="base_footprint_joint" type="fixed">
+      <parent link="base_footprint" />
+      <child link="base_link" />
+      <origin xyz="0 0 ${wheel_r}" rpy="0 0 0" />
     </joint>
+    <!-- Macro for defining wheels -->
+    <xacro:macro name="wheel" params="prefix reflect">
+      <link name="${prefix}_wheel">
+        <visual>
+          <origin xyz="${-0.071*reflect} 0 0" rpy="0 ${(reflect-1)*pi/2} 0" />
+          <geometry>
+            <mesh filename="package://magni_description/meshes/common/standard_wheel.dae" />
+          </geometry>
+        </visual>
+        <collision>
+          <origin xyz="0 0 0" rpy="0 ${pi/2} 0" />
+          <geometry>
+            <cylinder radius="${wheel_r}" length="0.05" />
+          </geometry>
+        </collision>
+        <collision>
+          <origin xyz="${0.033*reflect} 0 0" rpy="0 ${pi/2} 0" />
+          <geometry>
+            <cylinder radius="0.064" length="0.016" />
+          </geometry>
+        </collision>
+        <xacro:cylinder_inertial_with_origin radius="${wheel_r}" length="0.05" mass="3.34">
+          <origin xyz="0 0 0" rpy="0 ${pi/2} 0" />
+        </xacro:cylinder_inertial_with_origin>
+      </link>
+      <joint name="${prefix}_wheel_joint" type="continuous">
+        <axis xyz="1 0 0" rpy="0 0 0" />
+        <parent link="base_link" />
+        <child link="${prefix}_wheel" />
+        <origin xyz="0 ${0.163*reflect} 0" rpy="0 0 ${pi/2}" />
+      </joint>
+    </xacro:macro>
+    <xacro:wheel prefix="left" reflect="1" />
+    <xacro:wheel prefix="right" reflect="-1" />
+    <!-- Macro for defining caster wheels -->
+    <xacro:macro name="caster_wheel" params="prefix reflect">
+      <link name="${prefix}_caster_wheel">
+        <collision>
+          <origin xyz="${-wheel_xpos-0.19} ${reflect*0.169} ${-wheel_r+0.04}" rpy="0 0 0" />
+          <geometry>
+            <sphere radius="0.04" />
+          </geometry>
+        </collision>
+      </link>
+      <joint name="${prefix}_caster_wheel_joint" type="fixed">
+        <parent link="base_link" />
+        <child link="${prefix}_caster_wheel" />
+      </joint>
+    </xacro:macro>
+    <xacro:caster_wheel prefix="left" reflect="1" />
+    <xacro:caster_wheel prefix="right" reflect="-1" />
+    <!-- ROS 2 Control block -->
+    <ros2_control name="MagniSystem" type="system">
+      <hardware>
+        <!-- <xacro:if value="$(arg use_sim)">
+        <plugin>gz_ros2_control/GazeboSimSystem</plugin>
+      </xacro:if> -->
+        <xacro:unless value="$(arg use_sim)">
+          <plugin>ubiquity_motor_ros2/MotorHardware</plugin>
+        </xacro:unless>
+      </hardware>
+      <joint name="left_wheel_joint">
+        <command_interface name="velocity" />
+        <state_interface name="position" />
+        <state_interface name="velocity" />
+        <state_interface name="effort" />
+      </joint>
+      <joint name="right_wheel_joint">
+        <command_interface name="velocity" />
+        <state_interface name="position" />
+        <state_interface name="velocity" />
+        <state_interface name="effort" />
+      </joint>
+    </ros2_control>
+    <!-- Lidar Configuration for Mini (Top Plate) -->
+    <xacro:ur_c1_lidar name="laser" connected_to="base_link">
+      <origin xyz="-0.092 -0.066 0.23" rpy="0 0 0" />
+    </xacro:ur_c1_lidar>
   </xacro:macro>
-  <xacro:caster_wheel prefix="left" reflect="1"/>
-  <xacro:caster_wheel prefix="right" reflect="-1"/>
- <!-- ROS 2 Control block -->
-  <ros2_control name="MagniSystem" type="system">
-    <hardware>
-      <xacro:if value="$(arg use_sim)">
-        <plugin>gz_ros2_control/GazeboSimSystem</plugin>
-      </xacro:if>
-      <xacro:unless value="$(arg use_sim)">
-        <plugin>ubiquity_motor_ros2/MotorHardware</plugin>
-      </xacro:unless>
-    </hardware>
-    <joint name="left_wheel_joint">
-      <command_interface name="velocity"/>
-      <state_interface name="position"/>
-      <state_interface name="velocity"/>
-      <state_interface name="effort"/>
-    </joint>
-    <joint name="right_wheel_joint">
-      <command_interface name="velocity"/>
-      <state_interface name="position"/>
-      <state_interface name="velocity"/>
-      <state_interface name="effort"/>
-    </joint>
-  </ros2_control>
-  <!-- Lidar Configuration for Mini (Top Plate) -->
-  <xacro:ur_c1_lidar name="laser" connected_to="base_link">
-    <origin xyz="-0.092 -0.066 0.23" rpy="0 0 0"/>
-  </xacro:ur_c1_lidar>
 </robot>

Commit message: Added prefix for namespacing the gen 5 URDF

File: magni_description/urdf/robots/gen_5_silver.urdf.xacro (robot description, xacro)
@@ -2,5 +2,5 @@
 <robot xmlns:xacro="http://wiki.ros.org/xacro">
   <xacro:macro name="magni"
-    params="sonars_installed:=true shell_installed:=false tower_installed:=false camera_extrinsics_file:='' lidar_extrinsics_file:=''">
+    params="prefix:='' sonars_installed:=true shell_installed:=false tower_installed:=false camera_extrinsics_file:='' lidar_extrinsics_file:=''">
     <xacro:property name="wheel_r" value="0.1" />
     <xacro:property name="wheel_xpos" value="0.11" />
@@ -11,5 +11,5 @@
     <xacro:include filename="$(find magni_description)/urdf/sensors/ur_c1_lidar.xacro" />
     <!-- Robot base_link -->
-    <link name="base_link">
+    <link name="${prefix}base_link">
       <visual>
         <origin xyz="${-wheel_xpos} 0 ${-wheel_r+0.071}" rpy="0 0 0" />
@@ -119,13 +119,13 @@
     </link>
     <!-- Fixed offset from the floor to the center of the wheels -->
-    <link name="base_footprint" />
-    <joint name="base_footprint_joint" type="fixed">
-      <parent link="base_footprint" />
-      <child link="base_link" />
+    <link name="${prefix}base_footprint" />
+    <joint name="${prefix}base_footprint_joint" type="fixed">
+      <parent link="${prefix}base_footprint" />
+      <child link="${prefix}base_link" />
       <origin xyz="0 0 ${wheel_r}" rpy="0 0 0" />
     </joint>
     <!-- Macro for defining wheels -->
-    <xacro:macro name="wheel" params="prefix reflect">
-      <link name="${prefix}_wheel">
+    <xacro:macro name="wheel" params="wheel_prefix reflect">
+      <link name="${wheel_prefix}_wheel">
         <visual>
           <origin xyz="${-0.071*reflect} 0 0" rpy="0 ${(reflect-1)*pi/2} 0" />
@@ -150,16 +150,16 @@
         </xacro:cylinder_inertial_with_origin>
       </link>
-      <joint name="${prefix}_wheel_joint" type="continuous">
+      <joint name="${wheel_prefix}_wheel_joint" type="continuous">
         <axis xyz="1 0 0" rpy="0 0 0" />
-        <parent link="base_link" />
-        <child link="${prefix}_wheel" />
+        <parent link="${prefix}base_link" />
+        <child link="${wheel_prefix}_wheel" />
         <origin xyz="0 ${0.163*reflect} 0" rpy="0 0 ${pi/2}" />
       </joint>
     </xacro:macro>
-    <xacro:wheel prefix="left" reflect="1" />
-    <xacro:wheel prefix="right" reflect="-1" />
+    <xacro:wheel wheel_prefix="${prefix}left" reflect="1" />
+    <xacro:wheel wheel_prefix="${prefix}right" reflect="-1" />
     <!-- Macro for defining caster wheels -->
-    <xacro:macro name="caster_wheel" params="prefix reflect">
-      <link name="${prefix}_caster_wheel">
+    <xacro:macro name="caster_wheel" params="wheel_prefix reflect">
+      <link name="${wheel_prefix}_caster_wheel">
         <collision>
           <origin xyz="${-wheel_xpos-0.19} ${reflect*0.169} ${-wheel_r+0.04}" rpy="0 0 0" />
@@ -169,26 +169,26 @@
         </collision>
       </link>
-      <joint name="${prefix}_caster_wheel_joint" type="fixed">
-        <parent link="base_link" />
-        <child link="${prefix}_caster_wheel" />
+      <joint name="${wheel_prefix}_caster_wheel_joint" type="fixed">
+        <parent link="${prefix}base_link" />
+        <child link="${wheel_prefix}_caster_wheel" />
       </joint>
     </xacro:macro>
-    <xacro:caster_wheel prefix="left" reflect="1" />
-    <xacro:caster_wheel prefix="right" reflect="-1" />
+    <xacro:caster_wheel wheel_prefix="${prefix}left" reflect="1" />
+    <xacro:caster_wheel wheel_prefix="${prefix}right" reflect="-1" />
     <!-- Define all sonars, if sonars_installed set to 1 -->
     <xacro:if value="${sonars_installed}">
-      <xacro:sonar_hc-sr04 name="sonar_0" connected_to="base_link">
+      <xacro:sonar_hc-sr04 name="${prefix}sonar_0" connected_to="base_link">
         <origin xyz="0.01 -0.14 0.15" rpy="0 0 ${-pi/2}" />
       </xacro:sonar_hc-sr04>
-      <xacro:sonar_hc-sr04 name="sonar_1" connected_to="base_link">
+      <xacro:sonar_hc-sr04 name="${prefix}sonar_1" connected_to="base_link">
         <origin xyz="0.08 -0.07 0.15" rpy="0 0 0.785" />
       </xacro:sonar_hc-sr04>
-      <xacro:sonar_hc-sr04 name="sonar_2" connected_to="base_link">
+      <xacro:sonar_hc-sr04 name="${prefix}sonar_2" connected_to="base_link">
         <origin xyz="0.08 -0.01 0.15" rpy="0 0 -0.785" />
       </xacro:sonar_hc-sr04>
-      <xacro:sonar_hc-sr04 name="sonar_3" connected_to="base_link">
+      <xacro:sonar_hc-sr04 name="${prefix}sonar_3" connected_to="base_link">
         <origin xyz="0.08 0.04 0.15" rpy="0 0 0" />
       </xacro:sonar_hc-sr04>
-      <xacro:sonar_hc-sr04 name="sonar_4" connected_to="base_link">
+      <xacro:sonar_hc-sr04 name="${prefix}sonar_4" connected_to="base_link">
         <origin xyz="0.01 0.14 0.15" rpy="0 0 ${pi/2}" />
       </xacro:sonar_hc-sr04>
@@ -197,5 +197,5 @@
     <xacro:if value="${camera_extrinsics_file != ''}">
       <xacro:property name="cam_extrinsics" value="${xacro.load_yaml(camera_extrinsics_file)}" />
-      <xacro:raspi_camera name="raspicam" connected_to="base_link">
+      <xacro:raspi_camera name="${prefix}raspicam" connected_to="${prefix}base_link">
         <origin xyz="${cam_extrinsics['x']} ${cam_extrinsics['y']} ${cam_extrinsics['z']}"
           rpy="${cam_extrinsics['roll']} ${cam_extrinsics['pitch']} ${cam_extrinsics['yaw']}" />
@@ -205,5 +205,5 @@
     <xacro:if value="${lidar_extrinsics_file != ''}">
       <xacro:property name="lidar_extrinsics" value="${xacro.load_yaml(lidar_extrinsics_file)}" />
-      <xacro:ur_c1_lidar name="laser" connected_to="base_link">
+      <xacro:ur_c1_lidar name="${prefix}laser" connected_to="${prefix}base_link">
         <origin xyz="${lidar_extrinsics['x']} ${lidar_extrinsics['y']} ${lidar_extrinsics['z']}"
           rpy="${lidar_extrinsics['roll']} ${lidar_extrinsics['pitch']} ${lidar_extrinsics['yaw']}" />
@@ -215,5 +215,5 @@
         <plugin>ubiquity_motor_ros2/MotorHardware</plugin>
       </hardware>
-      <joint name="left_wheel_joint">
+      <joint name="${prefix}left_wheel_joint">
         <command_interface name="velocity" />
         <state_interface name="position" />
@@ -221,5 +221,5 @@
         <state_interface name="effort" />
       </joint>
-      <joint name="right_wheel_joint">
+      <joint name="${prefix}right_wheel_joint">
         <command_interface name="velocity" />
         <state_interface name="position" />

Commit message: Work toward gazebo sim

File: magni_description/urdf/robots/gen_5_silver.urdf.xacro (robot description, xacro)
@@ -144,4 +144,16 @@
         <origin xyz="0 ${0.163*reflect} 0" rpy="0 0 ${pi/2}" />
       </joint>
+      <gazebo reference="${wheel_prefix}_wheel">
+        <mu1 value="0.8"/>
+        <mu2 value="0.8"/>
+        <surface>
+          <friction>
+            <ode>
+              <mu>0.8</mu>
+              <mu2>0.8</mu2>
+            </ode>
+          </friction>
+        </surface>
+      </gazebo>
     </xacro:macro>
     <xacro:wheel wheel_prefix="${prefix}left" reflect="1" />
@@ -167,4 +179,16 @@
         <child link="${wheel_prefix}_caster_wheel" />
       </joint>
+      <gazebo reference="${wheel_prefix}_caster_wheel">
+        <mu1 value="0.0"/>
+        <mu2 value="0.0"/>
+        <surface>
+          <friction>
+            <ode>
+              <mu>0.0</mu>
+              <mu2>0.0</mu2>
+            </ode>
+          </friction>
+        </surface>
+      </gazebo>
     </xacro:macro>
     <xacro:caster_wheel wheel_prefix="${prefix}left" reflect="1" />
@@ -225,5 +249,5 @@
     </xacro:unless>
     <xacro:if value="${sim}">
-      <ros2_control name="GazeboSimSystem" type="system">
+      <ros2_control name="gz_ros2_control/GazeboSimSystem" type="system">
         <hardware>
           <plugin>gz_ros2_control/GazeboSimSystem</plugin>
@@ -243,5 +267,5 @@
       </ros2_control>
       <gazebo>
-        <plugin filename="gz_ros2_control-system" name="gz_ros2_control::GazeboSimROS2ControlPlugin">
+        <plugin filename="libgz_ros2_control-system.so" name="gz_ros2_control::GazeboSimROS2ControlPlugin">
           <parameters>${controller_config}</parameters>
         </plugin>
